File: pcb/kellorobo.sch (KiCad schematic (older format))
At the start: 12 parts, among them P1 Piezo, P2 Motor1, P3 Motor2, SW1 SW_PUSH, SW2 rotary_enc, U1 arduino_mini, U2 Ultra-hc-sr04, U3 l298n

Commit message: PCB ready with kicad. PCB svg files created for mill. Alignment, FCU, BCU and edges.
Parts:
- BT1: symbol Battery -> Battery-RESCUE-kellorobo
- D_LCD1: footprint Pin_Headers:Pin_Header_Angled_1x16 -> Pin_Headers:Pin_Header_Straight_1x16; symbol DISPLAY_HD44780 -> DISPLAY_HD44780-RESCUE-kellorobo
- RV1: footprint rotary_encoder_en11_hsb:rotary_encoder_EN11_HSB -> trimmeri:3165w-203p_trimmeri
Changed lines of the file:
@@
 EESchema Schematic File Version 2
+LIBS:kellorobo-rescue
 LIBS:power
 LIBS:device
@@
 LIBS:display_lcd
 LIBS:l298n
+LIBS:kellorobo-cache
 EELAYER 25 0
 EELAYER END
@@
 enb
 $Comp
-L DISPLAY_HD44780 D_LCD1
+L DISPLAY_HD44780-RESCUE-kellorobo D_LCD1
 U 1 1 57273D75
 P 10050 3900
 F 0 "D_LCD1" H 9050 4150 60  0000 C CNN
 F 1 "DISPLAY_HD44780" H 9800 4300 60  0000 C CNN
-F 2 "Pin_Headers:Pin_Header_Angled_1x16" H 10050 3900 60  0001 C CNN
+F 2 "Pin_Headers:Pin_Header_Straight_1x16" H 10050 3900 60  0001 C CNN
 F 3 "" H 10050 3900 60  0000 C CNN
 	1    10050 3900
@@
 F 0 "RV1" H 8850 4350 50  0000 C CNN
 F 1 "POT" H 8850 4450 50  0000 C CNN
-F 2 "rotary_encoder_en11_hsb:rotary_encoder_EN11_HSB" H 8850 4450 50  0001 C CNN
+F 2 "trimmeri:3165w-203p_trimmeri" H 8850 4450 50  0001 C CNN
 F 3 "" H 8850 4450 50  0000 C CNN
 	1    8850 4450
@@
 $EndComp
 $Comp
-L Battery BT1
+L Battery-RESCUE-kellorobo BT1
 U 1 1 57275D04
 P 3200 2000
